Commit message: Add duel observability and opponent tracking

File: src/sim_kobuki/description/kobuki.urdf.xacro (robot description, xacro)
@@ -3,4 +3,6 @@
   <xacro:arg name="ros_namespace" default="/"/>
   <xacro:arg name="frame_prefix" default=""/>
+  <xacro:arg name="lidar_horizontal_samples" default="900"/>
+  <xacro:arg name="lidar_vertical_samples" default="40"/>
   <xacro:property name="wheel_radius" value="0.035"/>
   <xacro:property name="wheel_width" value="0.0206"/>
@@ -180,4 +182,22 @@
     <mu2>1.2</mu2>
   </gazebo>
+  <!-- Gazebo-only body contact sensor for match evaluation. Wheels and floor
+       contacts are intentionally excluded. -->
+  <gazebo reference="base_link">
+    <sensor name="body_contact" type="contact">
+      <always_on>true</always_on>
+      <update_rate>20</update_rate>
+      <!-- Gazebo lumps base_link's fixed joint into base_footprint when the
+           URDF is spawned; this is the resulting collision name. -->
+      <contact><collision>base_footprint_fixed_joint_lump__base_link_collision</collision></contact>
+      <plugin name="body_bumper" filename="libgazebo_ros_bumper.so">
+        <ros>
+          <namespace>$(arg ros_namespace)</namespace>
+          <remapping>bumper_states:=body_contacts</remapping>
+        </ros>
+        <frame_name>$(arg frame_prefix)base_link</frame_name>
+      </plugin>
+    </sensor>
+  </gazebo>
   <gazebo reference="livox_frame">
     <!-- Пока штатный ray-лидар Gazebo Classic: вращательный паттерн, не
@@ -191,5 +211,5 @@
         <scan>
           <horizontal>
-            <samples>900</samples>
+            <samples>$(arg lidar_horizontal_samples)</samples>
             <resolution>1</resolution>
             <min_angle>-3.14159</min_angle>
@@ -197,5 +217,5 @@
           </horizontal>
           <vertical>
-            <samples>40</samples>
+            <samples>$(arg lidar_vertical_samples)</samples>
             <resolution>1</resolution>
             <min_angle>-0.1222</min_angle>  <!-- -7 град -->
