Commit message: Два робота в одном мире: защитник и атакующий
Первый шаг к дуэли: симулятор поднимает двух роботов, разведённых
пространствами имён, с независимым управлением и общим деревом TF. Логики
игры пока нет.

URDF параметризован аргументом ns. Пустое значение оставляет прежние имена,
поэтому одиночный запуск и maze.world работают как раньше. Заданное
разводит топики в /defender/... и фреймы в defender/odom. Префиксуются
только namespace плагинов и фреймы, которые они пишут в TF: имена link не
трогаются, так как robot_state_publisher добавляет frame_prefix сам.
frame_name у p3d остаётся world -- это общая для обоих система отсчёта.

Соперника каждый робот видит через TF, без детектирования лидаром. Оба
дерева одометрии подшиты к общему корню world статическим трансформом,
равным точке спавна, поэтому поза соперника берётся одним
lookup_transform. Это честно: odom по-прежнему ведёт diff_drive со своим
дрейфом, ground truth не подмешивается.

Роботы стартуют на площадках totami навстречу друг другу: защитник на синей
(3.5, 0) с yaw=pi, атакующий на красной (-3.5, 0).

Сервис duel отдельный, а не переключатель у gazebo: у них разные лаунчи и
разный набор аргументов. В профиль simulation не входит, так как каждый из
них поднимает свой gzserver.

Проверено: оба робота спавнятся, топики разведены, defender видит attacker
на 7.00 м, команда одному не двигает другого, RTF 1.00 и обе одометрии на
номинальных 50 Гц.

Co-Authored-By: Claude Opus 5 <noreply@anthropic.com>

File: src/sim_kobuki/description/kobuki.urdf.xacro (robot description, xacro)
@@ -5,4 +5,16 @@
        симулятора, облако не нужно. Включается через lidar:=true. -->
   <xacro:arg name="lidar" default="false"/>
+  <!-- Пространство имён робота. Пустое значение оставляет прежние имена
+       (/cmd_vel, /odom, фрейм odom) и один робот работает как раньше.
+       Заданное, например defender, разводит топики в /defender/... и фреймы
+       в defender/odom, чтобы несколько роботов в одном мире не мешали друг
+       другу.
+       Имена link внутри URDF не трогаем: robot_state_publisher добавляет к
+       ним frame_prefix сам. Префиксовать нужно только то, что плагины
+       Gazebo пишут в TF и в топики: они про namespace ничего не знают. -->
+  <xacro:arg name="ns" default=""/>
+  <xacro:property name="ns" value="$(arg ns)"/>
+  <xacro:property name="prefix" value="${ns + '/' if ns else ''}"/>
+  <xacro:property name="ros_ns" value="${'/' + ns if ns else '/'}"/>
   <xacro:property name="wheel_radius" value="0.035"/>
   <xacro:property name="wheel_width" value="0.0206"/>
@@ -219,9 +231,9 @@
       <plugin name="livox_lidar_controller" filename="libgazebo_ros_ray_sensor.so">
         <ros>
-          <namespace>/</namespace>
+          <namespace>${ros_ns}</namespace>
           <remapping>~/out:=livox/lidar</remapping>
         </ros>
         <output_type>sensor_msgs/PointCloud2</output_type>
-        <frame_name>livox_frame</frame_name>
+        <frame_name>${prefix}livox_frame</frame_name>
       </plugin>
     </sensor>
@@ -246,8 +258,8 @@
       <plugin name="livox_imu_controller" filename="libgazebo_ros_imu_sensor.so">
         <ros>
-          <namespace>/</namespace>
+          <namespace>${ros_ns}</namespace>
           <remapping>~/out:=livox/imu</remapping>
         </ros>
-        <frame_name>livox_frame</frame_name>
+        <frame_name>${prefix}livox_frame</frame_name>
       </plugin>
     </sensor>
@@ -256,5 +268,5 @@
     <plugin name="diff_drive_controller" filename="libgazebo_ros_diff_drive.so">
       <ros>
-        <namespace>/</namespace>
+        <namespace>${ros_ns}</namespace>
       </ros>
       <left_joint>wheel_left_joint</left_joint>
@@ -267,11 +279,11 @@
       <publish_odom_tf>true</publish_odom_tf>
       <publish_wheel_tf>false</publish_wheel_tf>
-      <odometry_frame>odom</odometry_frame>
-      <robot_base_frame>base_footprint</robot_base_frame>
+      <odometry_frame>${prefix}odom</odometry_frame>
+      <robot_base_frame>${prefix}base_footprint</robot_base_frame>
       <update_rate>50</update_rate>
     </plugin>
     <plugin name="joint_state_publisher" filename="libgazebo_ros_joint_state_publisher.so">
       <ros>
-        <namespace>/</namespace>
+        <namespace>${ros_ns}</namespace>
         <remapping>~/out:=joint_states</remapping>
       </ros>
@@ -288,5 +300,5 @@
     <plugin name="ground_truth_p3d" filename="libgazebo_ros_p3d.so">
       <ros>
-        <namespace>/</namespace>
+        <namespace>${ros_ns}</namespace>
         <remapping>odom:=localization/pose</remapping>
       </ros>
